File: pcb/rise/reclone-rise.sch (EAGLE design)
At the start: 0 parts

Commit message: Added board dimensions, holes, and a couple parts for microcontroller and FPGA
Parts:
- added MCU: STM32F407VGT6, reclone-rise:STM32F407VGT6
- added U1: 6SLX25FTG256, xilinx_devices_V6:6SLX25FTG256
- added USB: USB_A_2H, reclone-rise:USB_A_2H
